Commit message: Another fix of URDF and working table coordinate system

File: fanuc_experimental/fanuc_lrmate200id_support/urdf/lrmate200id_macro (copy).xacro (robot description, xacro)
@@ -178,5 +178,5 @@
     </joint>
     <joint name="${prefix}joint_2" type="revolute">
-      <origin xyz="0 0 0.047" rpy="0 0 0"/>
+      <origin xyz="0 0 0.050" rpy="0 0 0"/>
       <parent link="${prefix}link_1" />
       <child link="${prefix}link_2" />
@@ -185,5 +185,5 @@
     </joint>
     <joint name="${prefix}joint_3" type="revolute">
-      <origin xyz="0.0 0 0.257" rpy="0 0 0"/>
+      <origin xyz="0.0 0 0.275" rpy="0 0 0"/>
       <parent link="${prefix}link_2" />
       <child link="${prefix}link_3" />
@@ -192,5 +192,5 @@
     </joint>
     <joint name="${prefix}joint_4" type="revolute">
-      <origin xyz="0.06 0 0.02" rpy="0 0 0"/>
+      <origin xyz="0.06 0 0.01" rpy="0 0 0"/>
       <parent link="${prefix}link_3"/>
       <child link="${prefix}link_4"/>
