Commit message: New URDF, stl files for LRMate200iD4s

File: fanuc_experimental/fanuc_lrmate200id_support/urdf/lrmate200id_macro.xacro (robot description, xacro)
@@ -111,5 +111,5 @@
     <link name="${prefix}flange">
       <visual>
-        <origin xyz="0.006 0 0" rpy="0 0 0"/>
+        <origin xyz="0 0 0" rpy="0 0 0"/>
         <geometry>
           <mesh scale="0.001 0.001 0.001" filename="package://fanuc_lrmate200id_support/meshes/lrmate200id/visual/flange.stl"/>
@@ -126,5 +126,5 @@
     <link name="${prefix}gripper">
       <visual>
-        <origin xyz="0.006 0 0" rpy="0 0 -1.5708"/>
+        <origin xyz="0 0 0" rpy="0 0 0"/>
         <geometry>
           <mesh scale="0.001 0.001 0.001" filename="package://fanuc_lrmate200id_support/meshes/lrmate200id/visual/gripper.stl"/>
@@ -133,5 +133,5 @@
       </visual>
       <collision>
-        <origin xyz="0 0 0" rpy="0 0 -1.5708"/>
+        <origin xyz="0 0 0" rpy="0 0 0"/>
         <geometry>
           <mesh scale="0.001 0.001 0.001" filename="package://fanuc_lrmate200id_support/meshes/lrmate200id/collision/gripper.stl"/>
@@ -141,14 +141,14 @@
     <link name="${prefix}left_finger">
       <visual>
-        <origin xyz="0.088 -0.020 0" rpy="0 0 -1.5708"/>
-        <geometry>
-          <mesh scale="0.001 0.001 0.001" filename="package://fanuc_lrmate200id_support/meshes/lrmate200id/visual/finger.stl"/>
-        </geometry>
-        <xacro:material_fanuc_greyish />
-      </visual>
-      <collision>
-        <origin xyz="0.088 -0.020 0" rpy="0 3.14159 -1.5708"/>
-        <geometry>
-          <mesh scale="0.001 0.001 0.001" filename="package://fanuc_lrmate200id_support/meshes/lrmate200id/collision/finger.stl"/>
+        <origin xyz="0 0 0" rpy="0 0 0"/>
+        <geometry>
+          <mesh scale="0.001 0.001 0.001" filename="package://fanuc_lrmate200id_support/meshes/lrmate200id/visual/left_finger.stl"/>
+        </geometry>
+        <xacro:material_fanuc_greyish />
+      </visual>
+      <collision>
+        <origin xyz="0 0 0" rpy="0 0 0"/>
+        <geometry>
+          <mesh scale="0.001 0.001 0.001" filename="package://fanuc_lrmate200id_support/meshes/lrmate200id/collision/left_finger.stl"/>
         </geometry>
       </collision>
@@ -156,14 +156,14 @@
     <link name="${prefix}right_finger">
       <visual>
-        <origin xyz="0.088 0.020 0" rpy="0 3.14159 -1.5708"/>
-        <geometry>
-          <mesh scale="0.001 0.001 0.001" filename="package://fanuc_lrmate200id_support/meshes/lrmate200id/visual/finger.stl"/>
-        </geometry>
-        <xacro:material_fanuc_greyish />
-      </visual>
-      <collision>
-        <origin xyz="0.088 0.020 0" rpy="0 0 -1.5708"/>
-        <geometry>
-          <mesh scale="0.001 0.001 0.001" filename="package://fanuc_lrmate200id_support/meshes/lrmate200id/collision/finger.stl"/>
+        <origin xyz="0 0 0" rpy="0 0 0"/>
+        <geometry>
+          <mesh scale="0.001 0.001 0.001" filename="package://fanuc_lrmate200id_support/meshes/lrmate200id/visual/right_finger.stl"/>
+        </geometry>
+        <xacro:material_fanuc_greyish />
+      </visual>
+      <collision>
+        <origin xyz="0 0 0" rpy="0 0 0"/>
+        <geometry>
+          <mesh scale="0.001 0.001 0.001" filename="package://fanuc_lrmate200id_support/meshes/lrmate200id/collision/right_finger.stl"/>
         </geometry>
       </collision>
@@ -171,5 +171,5 @@
     <!-- joints: main serial chain -->
     <joint name="${prefix}joint_1" type="revolute">
-      <origin xyz="0 0 0.330" rpy="0 0 0" />
+      <origin xyz="0 0 0.290" rpy="0 0 0" />
       <parent link="${prefix}base_link" />
       <child link="${prefix}link_1" />
@@ -178,5 +178,5 @@
     </joint>
     <joint name="${prefix}joint_2" type="revolute">
-      <origin xyz="0.050 0 0" rpy="0 0 0"/>
+      <origin xyz="0 0 0.050" rpy="0 0 0"/>
       <parent link="${prefix}link_1" />
       <child link="${prefix}link_2" />
@@ -185,5 +185,5 @@
     </joint>
     <joint name="${prefix}joint_3" type="revolute">
-      <origin xyz="0 0 0.330" rpy="0 0 0"/>
+      <origin xyz="0.0 0 0.275" rpy="0 0 0"/>
       <parent link="${prefix}link_2" />
       <child link="${prefix}link_3" />
@@ -192,5 +192,5 @@
     </joint>
     <joint name="${prefix}joint_4" type="revolute">
-      <origin xyz="0 0 0.035" rpy="0 0 0"/>
+      <origin xyz="0.06 0 0.01" rpy="0 0 0"/>
       <parent link="${prefix}link_3"/>
       <child link="${prefix}link_4"/>
@@ -199,5 +199,5 @@
     </joint>
     <joint name="${prefix}joint_5" type="revolute">
-      <origin xyz="0.335 0 0" rpy="0 0 0"/>
+      <origin xyz="0.226 0 0" rpy="0 0 0"/>
       <parent link="${prefix}link_4"/>
       <child link="${prefix}link_5"/>
@@ -206,5 +206,5 @@
     </joint>
     <joint name="${prefix}joint_6" type="revolute">
-      <origin xyz="0.080 0 0" rpy="0 0 0"/>
+      <origin xyz="0.040 0 0" rpy="0 0 0"/>
       <parent link="${prefix}link_5"/>
       <child link="${prefix}link_6"/>
@@ -215,5 +215,5 @@
     <link name="${prefix}base" />
     <joint name="${prefix}base_link-base" type="fixed">
-      <origin xyz="0 0 0.330" rpy="0 0 0"/>
+      <origin xyz="0 0 0.290" rpy="0 0 0"/>
       <parent link="${prefix}base_link"/>
       <child link="${prefix}base"/>
@@ -222,5 +222,5 @@
     <!--<link name="${prefix}flange" />-->
     <joint name="${prefix}joint_6-flange" type="fixed">
-      <origin xyz="0 0 0" rpy="0 0 0" />
+      <origin xyz="0.038 0.0 0.0" rpy="0 0 0" />
       <parent link="${prefix}link_6" />
       <child link="${prefix}flange" />
@@ -229,5 +229,5 @@
     <joint name="${prefix}flange-gripper" type="fixed">
       <!--<origin xyz="0 0 0" rpy="${pi} ${-pi/2.0} 0" />-->
-      <origin xyz="0 0 0" rpy="0 0 0" />
+      <origin xyz="0.012 0 0" rpy="0 0 0" />
       <parent link="${prefix}flange" />
       <child link="${prefix}gripper" />
@@ -236,5 +236,5 @@
         <parent link="gripper" />
         <child link="left_finger" />
-        <origin rpy="0 0 0" xyz="0 0 0" />
+        <origin xyz="0.088 0 0" rpy="0 0 0" />
         <axis xyz="0 1 0" />
         <limit effort="20" lower="0.0" upper="0.04" velocity="0.2" />
@@ -243,5 +243,5 @@
         <parent link="gripper" />
         <child link="right_finger" />
-        <origin rpy="0 0 0" xyz="0 0 0" />
+        <origin xyz="0.088 0 0" rpy="0 0 0" />
         <axis xyz="0 -1 0" />
         <limit effort="20" lower="0.0" upper="0.04" velocity="0.2" />

Commit message: Putting tool0 frame back, offsets of joint1 to match the real robot

File: fanuc_experimental/fanuc_lrmate200id_support/urdf/lrmate200id_macro.xacro (robot description, xacro)
@@ -96,5 +96,5 @@
     <link name="${prefix}link_6">
       <visual>
-        <origin xyz="0 0 0" rpy="0 0 0"/>
+        <origin xyz="-0.057 0 0" rpy="0 0 0"/>
         <geometry>
           <mesh filename="package://fanuc_lrmate200id_support/meshes/lrmate200id/visual/link_6.stl"/>
@@ -109,20 +109,20 @@
       </collision>
     </link>
+    <!--<link name="${prefix}flange">
+      <visual>
+        <origin xyz="0 0 0" rpy="0 0 0"/>
+        <geometry>
+          <mesh scale="0.001 0.001 0.001" filename="package://fanuc_lrmate200id_support/meshes/lrmate200id/visual/flange.stl"/>
+        </geometry>
+        <xacro:material_fanuc_greyish />
+      </visual>
+      <collision>
+        <origin xyz="0 0 0" rpy="0 0 0"/>
+        <geometry>
+          <mesh scale="0.001 0.001 0.001" filename="package://fanuc_lrmate200id_support/meshes/lrmate200id/collision/flange.stl"/>
+        </geometry>
+      </collision>
+    </link>-->
     <link name="${prefix}flange">
-      <visual>
-        <origin xyz="0 0 0" rpy="0 0 0"/>
-        <geometry>
-          <mesh scale="0.001 0.001 0.001" filename="package://fanuc_lrmate200id_support/meshes/lrmate200id/visual/flange.stl"/>
-        </geometry>
-        <xacro:material_fanuc_greyish />
-      </visual>
-      <collision>
-        <origin xyz="0 0 0" rpy="0 0 0"/>
-        <geometry>
-          <mesh scale="0.001 0.001 0.001" filename="package://fanuc_lrmate200id_support/meshes/lrmate200id/collision/flange.stl"/>
-        </geometry>
-      </collision>
-    </link>
-    <link name="${prefix}gripper">
       <visual>
         <origin xyz="0 0 0" rpy="0 0 0"/>
@@ -171,5 +171,5 @@
     <!-- joints: main serial chain -->
     <joint name="${prefix}joint_1" type="revolute">
-      <origin xyz="0 0 0.290" rpy="0 0 0" />
+      <origin xyz="-0.006 -0.002 0.290" rpy="0 0 0" />
       <parent link="${prefix}base_link" />
       <child link="${prefix}link_1" />
@@ -178,5 +178,5 @@
     </joint>
     <joint name="${prefix}joint_2" type="revolute">
-      <origin xyz="0 0 0.047" rpy="0 0 0"/>
+      <origin xyz="0 0 0.040" rpy="0 0 0"/>
       <parent link="${prefix}link_1" />
       <child link="${prefix}link_2" />
@@ -185,5 +185,5 @@
     </joint>
     <joint name="${prefix}joint_3" type="revolute">
-      <origin xyz="0.0 0 0.257" rpy="0 0 0"/>
+      <origin xyz="0.0 0 0.26" rpy="0 0 0"/>
       <parent link="${prefix}link_2" />
       <child link="${prefix}link_3" />
@@ -192,5 +192,5 @@
     </joint>
     <joint name="${prefix}joint_4" type="revolute">
-      <origin xyz="0.06 0 0.02" rpy="0 0 0"/>
+      <origin xyz="0.064 0 0.02" rpy="0 0 0"/>
       <parent link="${prefix}link_3"/>
       <child link="${prefix}link_4"/>
@@ -206,5 +206,5 @@
     </joint>
     <joint name="${prefix}joint_6" type="revolute">
-      <origin xyz="0.040 0 0" rpy="0 0 0"/>
+      <origin xyz="0.070 0 0" rpy="0 0 0"/>
       <parent link="${prefix}link_5"/>
       <child link="${prefix}link_6"/>
@@ -222,28 +222,34 @@
     <!--<link name="${prefix}flange" />-->
     <joint name="${prefix}joint_6-flange" type="fixed">
-      <origin xyz="0.038 0.0 0.0" rpy="0 0 0" />
+      <origin xyz="0.0 0.0 0.0" rpy="0 0 0" />
       <parent link="${prefix}link_6" />
       <child link="${prefix}flange" />
     </joint>
     <!-- Schunk gripper frame -->
-    <joint name="${prefix}flange-gripper" type="fixed">
-      <!--<origin xyz="0 0 0" rpy="${pi} ${-pi/2.0} 0" />-->
-      <origin xyz="0.012 0 0" rpy="0 0 0" />
+    <!--<joint name="${prefix}flange-gripper" type="fixed">
+      <origin xyz="0.0 0 0" rpy="0 0 0" />
       <parent link="${prefix}flange" />
       <child link="${prefix}gripper" />
+    </joint>-->
+    <!-- ROS-Industrial 'tool0' frame: all-zeros tool frame -->
+    <link name="${prefix}tool0" />
+    <joint name="${prefix}link_6-tool0" type="fixed">
+      <origin xyz="0.13 0 0" rpy="${pi} ${-pi/2.0} 0" />
+      <parent link="${prefix}link_6" />
+      <child link="${prefix}tool0" />
     </joint>
     <joint name="finger_joint1" type="prismatic">
-        <parent link="gripper" />
+        <parent link="flange" />
         <child link="left_finger" />
+        <origin xyz="0.088 0 0" rpy="0 0 0" />
+        <axis xyz="0 -1 0" />
+        <limit effort="20" lower="0.0" upper="0.04" velocity="0.2" />
+    </joint>
+    <joint name="finger_joint2" type="prismatic">
+        <parent link="flange" />
+        <child link="right_finger" />
         <origin xyz="0.088 0 0" rpy="0 0 0" />
         <axis xyz="0 1 0" />
         <limit effort="20" lower="0.0" upper="0.04" velocity="0.2" />
-    </joint>
-    <joint name="finger_joint2" type="prismatic">
-        <parent link="gripper" />
-        <child link="right_finger" />
-        <origin xyz="0.088 0 0" rpy="0 0 0" />
-        <axis xyz="0 -1 0" />
-        <limit effort="20" lower="0.0" upper="0.04" velocity="0.2" />
         <mimic joint="finger_joint1" />
     </joint>
